File: v1 4 button.brd (EAGLE design)
At the start: 45 x 80 mm, 31 parts, among them IC5 AMS1117-3.3V, X1 0446200002

Commit message: Add files via upload
Parts:
- C5: device rcl:UD-6,3X7,7_NICHICON -> rcl:UD-10X10_NICHICON
- moved C5 1.00 mm to (6.50, 71.0)
Routing:
- net GND: track 117.3 -> 119.8 mm
Changed lines of the file:
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@@
 <attribute name="VALUE" x="28.5" y="54.5" size="1.27" layer="27" rot="R180"/>
 </element>
-<element name="C5" library="rcl" library_urn="urn:adsk.eagle:library:334" package="UD-6,3X7,7_NICHICON" package3d_urn="urn:adsk.eagle:package:23472/1" value="1000uf" x="6.5" y="70" smashed="yes" rot="R90">
-<attribute name="NAME" x="2.69" y="66.825" size="1.016" layer="25" rot="R90"/>
-<attribute name="POPULARITY" value="1" x="47.14" y="106.83" size="1.778" layer="27" rot="R90" display="off"/>
-<attribute name="SPICEPREFIX" value="C" x="47.14" y="106.83" size="1.778" layer="27" rot="R90" display="off"/>
-<attribute name="VALUE" x="10.945" y="66.825" size="1.016" layer="27" rot="R90"/>
+<element name="C5" library="rcl" library_urn="urn:adsk.eagle:library:334" package="UD-10X10_NICHICON" package3d_urn="urn:adsk.eagle:package:23469/1" value="1000uf" x="6.5" y="71" smashed="yes" rot="R90">
+<attribute name="NAME" x="2.69" y="67.825" size="1.016" layer="25" rot="R90"/>
+<attribute name="POPULARITY" value="1" x="47.14" y="107.83" size="1.778" layer="27" rot="R90" display="off"/>
+<attribute name="SPICEPREFIX" value="C" x="47.14" y="107.83" size="1.778" layer="27" rot="R90" display="off"/>
+<attribute name="VALUE" x="10.945" y="67.825" size="1.016" layer="27" rot="R90"/>
 </element>
 <element name="C6" library="rcl" library_urn="urn:adsk.eagle:library:334" package="C0603" package3d_urn="urn:adsk.eagle:package:23616/2" value="0.1uf" x="37.5" y="75" smashed="yes" rot="R90">
@@
 <wire x1="41.5" y1="76.849" x2="41.5" y2="71" width="1.27" layer="1"/>
 <wire x1="41.5" y1="76.849" x2="40" y2="78.349" width="1.27" layer="1"/>
-<wire x1="40" y1="78.349" x2="9.849" y2="78.349" width="1.27" layer="1"/>
+<wire x1="40" y1="78.349" x2="8.849" y2="78.349" width="1.27" layer="1"/>
 <wire x1="37.5" y1="69.5" x2="40" y2="69.5" width="1.27" layer="1"/>
-<wire x1="6.5" y1="75" x2="6.5" y2="72.35" width="1.27" layer="1"/>
-<wire x1="9.849" y1="78.349" x2="6.5" y2="75" width="1.27" layer="1"/>
-<via x="6.5" y="75" extent="1-16" drill="0.35"/>
-<wire x1="6.5" y1="75" x2="1.651" y2="70.151" width="1.27" layer="16"/>
+<wire x1="5.575" y1="74" x2="4.5" y2="74" width="1.27" layer="1"/>
+<wire x1="5.575" y1="74" x2="6.5" y2="74.925" width="1.27" layer="1"/>
+<wire x1="8.849" y1="78.349" x2="4.5" y2="74" width="1.27" layer="1"/>
+<via x="4.5" y="74" extent="1-16" drill="0.35"/>
+<wire x1="4.5" y1="74" x2="4.5" y2="73.5" width="1.27" layer="16"/>
+<wire x1="4.5" y1="73.5" x2="1.651" y2="70.651" width="1.27" layer="16"/>
 <wire x1="1.651" y1="7.5" x2="7.5" y2="1.651" width="1.27" layer="16"/>
 <wire x1="7.5" y1="1.651" x2="8" y2="1.651" width="1.27" layer="16"/>
 <wire x1="8" y1="1.651" x2="16" y2="1.651" width="1.27" layer="16"/>
 <wire x1="16" y1="1.651" x2="18.5" y2="4.151" width="1.27" layer="16"/>
-<wire x1="1.651" y1="70.151" x2="1.651" y2="64" width="1.27" layer="16"/>
+<wire x1="1.651" y1="70.651" x2="1.651" y2="64" width="1.27" layer="16"/>
 <wire x1="1.651" y1="64" x2="1.651" y2="56.5" width="1.27" layer="16"/>
 <wire x1="1.651" y1="56.5" x2="1.651" y2="46" width="1.27" layer="16"/>
@@
 <wire x1="18.161" y1="49.1744" x2="18.11629375" y2="49.212134375" width="0.4064" layer="1"/>
 <wire x1="29.337" y1="46.6598" x2="29.712134375" y2="46.38370625" width="0.4064" layer="1"/>
+<wire x1="42.11629375" y1="49.212134375" x2="42.11629375" y2="49.21213125" width="0" layer="19" extent="1-1"/>
+<wire x1="26.883703125" y1="58.787865625" x2="26.88370625" y2="58.787865625" width="0" layer="19" extent="1-1"/>
+<wire x1="18.11629375" y1="49.21213125" x2="18.11629375" y2="49.212134375" width="0" layer="19" extent="1-1"/>
+<wire x1="5.71213125" y1="46.383703125" x2="5.712134375" y2="46.38370625" width="0" layer="19" extent="1-1"/>
+<wire x1="42.11629375" y1="5.21213125" x2="42.11629375" y2="5.212134375" width="0" layer="19" extent="1-1"/>
+<wire x1="29.71213125" y1="2.383703125" x2="29.712134375" y2="2.38370625" width="0" layer="19" extent="1-1"/>
+<wire x1="18.11629375" y1="5.21213125" x2="18.11629375" y2="5.212134375" width="0" layer="19" extent="1-1"/>
+<wire x1="5.71213125" y1="2.383703125" x2="5.712134375" y2="2.38370625" width="0" layer="19" extent="1-1"/>
+<wire x1="2.883703125" y1="58.787865625" x2="1.651" y2="56.5" width="0" layer="19" extent="1-1"/>
+<wire x1="2.883703125" y1="14.787865625" x2="1.651" y2="12.5" width="0" layer="19" extent="1-1"/>
+<wire x1="29.71213125" y1="46.383703125" x2="32.5" y2="46" width="0" layer="19" extent="1-1"/>
+<wire x1="26.883703125" y1="14.787865625" x2="26.5" y2="12" width="0" layer="19" extent="1-1"/>
 </signal>
 <signal name="GND">
@@
 <wire x1="39.5" y1="75" x2="39.5" y2="73.06" width="1.27" layer="1"/>
 <via x="38.65" y="75.85" extent="1-16" drill="0.35"/>
-<wire x1="6.5" y1="67.65" x2="6.65" y2="67.65" width="1.27" layer="1"/>
-<wire x1="6.65" y1="67.65" x2="8" y2="69" width="1.27" layer="1"/>
-<via x="8" y="69" extent="1-16" drill="0.35"/>
+<wire x1="6.5" y1="67.05" x2="6.650003125" y2="68.650003125" width="1.27" layer="1"/>
+<wire x1="8" y1="70" x2="8" y2="71" width="1.27" layer="1"/>
+<wire x1="8" y1="70" x2="6.650003125" y2="68.650003125" width="1.27" layer="1"/>
+<via x="8" y="71" extent="1-16" drill="0.35"/>
 <wire x1="5.28786875" y1="51.616296875" x2="6.5" y2="52.828428125" width="1.016" layer="1"/>
 <wire x1="6.5" y1="52.828428125" x2="6.5" y2="53.15" width="1.016" layer="1"/>
@@
 <vertex x="39" y="80"/>
 </polygon>
+<wire x1="25.556" y1="71.318" x2="33.5" y2="75.85" width="0" layer="19" extent="1-1"/>
+<wire x1="32.11629375" y1="59.21213125" x2="24.54" y2="69.54" width="0" layer="19" extent="1-1"/>
+<wire x1="32.116296875" y1="59.21213125" x2="32.11629375" y2="59.21213125" width="0" layer="19" extent="1-1"/>
+<wire x1="36.883703125" y1="48.787865625" x2="36.883703125" y2="48.78786875" width="0" layer="19" extent="1-1"/>
+<wire x1="29.287865625" y1="51.61629375" x2="29.28786875" y2="51.616296875" width="0" layer="19" extent="1-1"/>
+<wire x1="30.215" y1="43.43" x2="29.28786875" y2="51.616296875" width="0" layer="19" extent="1-1"/>
+<wire x1="15.71213125" y1="56.383703125" x2="29.28786875" y2="51.616296875" width="0" layer="19" extent="1-1"/>
+<wire x1="8.11629375" y1="59.21213125" x2="8.116296875" y2="59.21213125" width="0" layer="19" extent="1-1"/>
+<wire x1="12.883703125" y1="48.787865625" x2="12.883703125" y2="48.78786875" width="0" layer="19" extent="1-1"/>
+<wire x1="5.287865625" y1="51.61629375" x2="5.28786875" y2="51.616296875" width="0" layer="19" extent="1-1"/>
+<wire x1="6.5" y1="67.05" x2="8.116296875" y2="59.21213125" width="0" layer="19" extent="1-1"/>
+<wire x1="32.11629375" y1="15.21213125" x2="30.215" y2="43.43" width="0" layer="19" extent="1-1"/>
+<wire x1="32.116296875" y1="15.21213125" x2="32.11629375" y2="15.21213125" width="0" layer="19" extent="1-1"/>
+<wire x1="36.883703125" y1="4.787865625" x2="36.883703125" y2="4.78786875" width="0" layer="19" extent="1-1"/>
+<wire x1="29.287865625" y1="7.61629375" x2="29.28786875" y2="7.616296875" width="0" layer="19" extent="1-1"/>
+<wire x1="15.71213125" y1="12.383703125" x2="29.28786875" y2="7.616296875" width="0" layer="19" extent="1-1"/>
+<wire x1="8.11629375" y1="15.21213125" x2="8.116296875" y2="15.21213125" width="0" layer="19" extent="1-1"/>
+<wire x1="12.883703125" y1="4.787865625" x2="12.883703125" y2="4.78786875" width="0" layer="19" extent="1-1"/>
+<wire x1="5.287865625" y1="7.61629375" x2="5.28786875" y2="7.616296875" width="0" layer="19" extent="1-1"/>
 </signal>
 <signal name="N$2">
