File: v2 4 button.brd (EAGLE design)
At the start: 45 x 80 mm, 23 parts, among them IC5 AMS1117-3.3V, J1 PTS636_SM25F_SMTR_LFS, J2 PTS636_SM25F_SMTR_LFS, J3 PTS636_SM25F_SMTR_LFS, J4 PTS636_SM25F_SMTR_LFS, J5 PTS636_SM25F_SMTR_LFS, J6 PTS636_SM25F_SMTR_LFS, J7 PTS636_SM25F_SMTR_LFS, J8 PTS636_SM25F_SMTR_LFS, X1 0446200002

Commit message: Add files via upload
Parts:
- C5: device rcl:UD-6,3X7,7_NICHICON -> rcl:UD-10X10_NICHICON
Routing:
- net VCC: track 215.2 -> 213.6 mm
- net GND: track 78.8 -> 80.1 mm
Changed lines of the file:
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@@
 <attribute name="VALUE" x="28" y="54" size="1.27" layer="27" rot="R180"/>
 </element>
-<element name="C5" library="rcl" library_urn="urn:adsk.eagle:library:334" package="UD-6,3X7,7_NICHICON" package3d_urn="urn:adsk.eagle:package:23472/1" value="1000uf" x="6.5" y="70" smashed="yes" rot="R90">
+<element name="C5" library="rcl" library_urn="urn:adsk.eagle:library:334" package="UD-10X10_NICHICON" package3d_urn="urn:adsk.eagle:package:23469/1" value="1000uf" x="6.5" y="70" smashed="yes" rot="R90">
 <attribute name="NAME" x="2.69" y="66.825" size="1.016" layer="25" rot="R90"/>
 <attribute name="POPULARITY" value="1" x="47.14" y="87.78" size="1.778" layer="27" rot="R90" display="off"/>
@@
 <wire x1="34" y1="48.5" x2="36.5" y2="51" width="1.27" layer="1"/>
 <wire x1="36.5" y1="51" x2="36.5" y2="52.3" width="1.27" layer="1"/>
-<wire x1="6.5" y1="67.65" x2="6.5" y2="65.5" width="1.27" layer="1"/>
-<via x="6.5" y="65.5" extent="1-16" drill="0.35"/>
+<wire x1="6.5" y1="66.05" x2="8.5" y2="64.05" width="1.27" layer="1"/>
+<wire x1="8.5" y1="64.05" x2="8.5" y2="63.5" width="1.27" layer="1"/>
+<via x="8.5" y="63.5" extent="1-16" drill="0.35"/>
 <polygon width="0.127" layer="16">
 <vertex x="5" y="80" curve="90"/>
@@
 <wire x1="35.7632" y1="75.9968" x2="35.7632" y2="75.85" width="0.4064" layer="1"/>
 <via x="35.7632" y="75.9968" extent="1-16" drill="0.35"/>
+<wire x1="25.556" y1="71.318" x2="33.5" y2="75.85" width="0" layer="19" extent="1-1"/>
+<wire x1="29" y1="59" x2="24.54" y2="69.54" width="0" layer="19" extent="1-1"/>
+<wire x1="29.5" y1="53.15" x2="29" y2="59" width="0" layer="19" extent="1-1"/>
+<wire x1="29.935" y1="43.52" x2="29" y2="48" width="0" layer="19" extent="1-1"/>
+<wire x1="12.5" y1="52.3" x2="29.5" y2="53.15" width="0" layer="19" extent="1-1"/>
+<wire x1="5" y1="59" x2="6" y2="53.15" width="0" layer="19" extent="1-1"/>
+<wire x1="8.5" y1="63.5" x2="7.2" y2="59" width="0" layer="19" extent="1-1"/>
+<wire x1="29" y1="15" x2="29.935" y2="43.52" width="0" layer="19" extent="1-1"/>
+<wire x1="30" y1="9.15" x2="29" y2="15" width="0" layer="19" extent="1-1"/>
+<wire x1="13" y1="8.3" x2="29" y2="5" width="0" layer="19" extent="1-1"/>
+<wire x1="5.5" y1="15" x2="6.5" y2="9.15" width="0" layer="19" extent="1-1"/>
 </signal>
 <signal name="B1">
@@
 <wire x1="42" y1="75.849" x2="39.5" y2="78.349" width="1.27" layer="1"/>
 <wire x1="39.5" y1="78.349" x2="8.349" y2="78.349" width="1.27" layer="1"/>
-<wire x1="6.5" y1="76.5" x2="6.5" y2="72.35" width="1.27" layer="1"/>
+<wire x1="6.5" y1="76.5" x2="6.5" y2="73.925" width="1.27" layer="1"/>
 <wire x1="37.5" y1="69" x2="40" y2="69" width="1.27" layer="1"/>
 <wire x1="42" y1="71" x2="42" y2="75.849" width="1.27" layer="1"/>
