File: v2 4 button.sch (EAGLE design)
At the start: 23 parts, among them IC5 AMS1117-3.3V, J1 PTS636_SM25F_SMTR_LFS, J2 PTS636_SM25F_SMTR_LFS, J3 PTS636_SM25F_SMTR_LFS, J4 PTS636_SM25F_SMTR_LFS, J5 PTS636_SM25F_SMTR_LFS, J6 PTS636_SM25F_SMTR_LFS, J7 PTS636_SM25F_SMTR_LFS, J8 PTS636_SM25F_SMTR_LFS, X1 0446200002

Commit message: Add files via upload
Parts:
- C5: device rcl:CPOL-EUUD-6,3X7,7 -> rcl:CPOL-USUD-10X10
Changed lines of the file:
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@@
 <part name="C3" library="rcl" library_urn="urn:adsk.eagle:library:334" deviceset="C-EU" device="C0603" package3d_urn="urn:adsk.eagle:package:23616/2" value="0.1uf"/>
 <part name="C4" library="rcl" library_urn="urn:adsk.eagle:library:334" deviceset="C-EU" device="C0603" package3d_urn="urn:adsk.eagle:package:23616/2" value="0.1uf"/>
-<part name="C5" library="rcl" library_urn="urn:adsk.eagle:library:334" deviceset="CPOL-EU" device="UD-6,3X7,7" package3d_urn="urn:adsk.eagle:package:23472/1" value="1000uf"/>
+<part name="C5" library="rcl" library_urn="urn:adsk.eagle:library:334" deviceset="CPOL-US" device="UD-10X10" package3d_urn="urn:adsk.eagle:package:23469/1" value="1000uf"/>
 <part name="IC5" library="SamacSys_Parts" deviceset="AMS1117-3.3V" device=""/>
 <part name="C6" library="rcl" library_urn="urn:adsk.eagle:library:334" deviceset="C-EU" device="C0603" package3d_urn="urn:adsk.eagle:package:23616/2" value="0.1uf"/>
