File: version 2/v2/v2 4 button.brd (EAGLE design)
At the start: 45 x 63.5 mm, 23 parts, among them IC5 AMS1117-3.3V, J1 PTS636_SM25F_SMTR_LFS, J2 PTS636_SM25F_SMTR_LFS, J3 PTS636_SM25F_SMTR_LFS, J4 PTS636_SM25F_SMTR_LFS, J5 PTS636_SM25F_SMTR_LFS, J6 PTS636_SM25F_SMTR_LFS, J7 PTS636_SM25F_SMTR_LFS, J8 PTS636_SM25F_SMTR_LFS, X1 0446200002

Commit message: Add files via upload
Parts:
- added D1, D2, D3, D4: SM4007PL, SamacSys_Parts:SODFL3718X125N
- added J9: (no value), SparkFun-Connectors:SCREWTERMINAL-5MM-2
- added SJ1: (no value), SparkFun-Retired:SJ_3_PASTE1&2
- added U$2: LOGO, custom parts:LOGO
- C5: device rcl:UD-10X10_NICHICON -> SamacSys_Parts:CAPAE1030X1050N
- X1: device con-molex:0446200002 -> custom parts:0446200002
- moved C6 12.2 mm to (33.5, 47.0), turned to 0 degrees
- moved C7 8.56 mm to (32.5, 50.0)
- moved IC5 1.00 mm to (37.5, 52.5)
- turned C5 to 270 degrees
Connections:
- new net D1-B1: D1.2, U$1.JP1.4
- new net D1-B2: D2.2, U$1.JP1.5
- new net D1-B3: D3.2, U$1.JP1.6
- new net D1-B4: D4.2, U$1.JP1.7
- new net N$4: SJ1.1, X1.4, X1.5
- new net N$6: J9.2, SJ1.3
- net B1: now also D1.1; no longer U$1.JP1.4
- net B2: now also D2.1; no longer U$1.JP1.5
- net B3: now also D3.1; no longer U$1.JP1.6
- net B4: now also D4.1; no longer U$1.JP1.7
- net GND: now also C5.2, J9.1; no longer C5.-
- net VCC: now also C5.1, IC5.4; no longer C5.+
- net VDD: now also SJ1.2; no longer X1.4, X1.5
Routing:
- net LED: track 41.9 -> 19.5 mm, vias 1 -> 2
- net N$6: track 0.00 -> 13.2 mm
- net N$4: track 0.00 -> 11.5 mm
- net GND: track 79.0 -> 88.8 mm, vias 10 -> 9
- net B3: track 59.8 -> 52.3 mm
- net D1-B4: track 0.00 -> 6.67 mm
- net B4: track 103.1 -> 97.5 mm
- net D1-B2: track 0.00 -> 5.15 mm
- net D1-B3: track 0.00 -> 5.13 mm
- net B1: track 59.7 -> 55.2 mm
- net D1-B1: track 0.00 -> 4.37 mm
- net N$5: track 18.8 -> 22.6 mm
- net VDD: track 22.0 -> 18.7 mm
- net VCC: track 183.0 -> 184.4 mm
- net B2: track 89.0 -> 88.8 mm, vias 1 -> 4
Other:
- board text added: "+ -"
- board text added: "7-30v"
- board text added: "V0.0.3"
