File: version 2/v2/v2 4 button.sch (EAGLE design)
At the start: 23 parts, among them IC5 AMS1117-3.3V, J1 PTS636_SM25F_SMTR_LFS, J2 PTS636_SM25F_SMTR_LFS, J3 PTS636_SM25F_SMTR_LFS, J4 PTS636_SM25F_SMTR_LFS, J5 PTS636_SM25F_SMTR_LFS, J6 PTS636_SM25F_SMTR_LFS, J7 PTS636_SM25F_SMTR_LFS, J8 PTS636_SM25F_SMTR_LFS, X1 0446200002

Commit message: Add files via upload
Parts:
- added D1, D2, D3, D4: SM4007PL, SamacSys_Parts:SM4007PL
- added J9: (no value), SparkFun-Connectors:CONN_025MM
- added SJ1: (no value), SparkFun-Retired:SOLDERJUMPER_2WAYPASTE1&2
- added U$2: LOGO, custom parts:LOGO
- C5: device rcl:CPOL-USUD-10X10 -> SamacSys_Parts:EEE-0JA102P
- X1: device con-molex:0446200002 -> custom parts:0446200002
Connections:
- new net D1-B1: D1.A, U$1.D5
- new net D1-B2: D2.A, U$1.D6
- new net D1-B3: D3.A, U$1.D7
- new net D1-B4: D4.A, U$1.D8
- new net N$4: SJ1.1, X1.4, X1.5
- new net N$6: J9.2, SJ1.3
- net B1: now also D1.K; no longer U$1.D5
- net B2: now also D2.K; no longer U$1.D6
- net B3: now also D3.K; no longer U$1.D7
- net B4: now also D4.K; no longer U$1.D8
- net GND: now also J9.1
- net VCC: now also IC5.OUTPUT
- net VDD: now also SJ1.2; no longer X1.4, X1.5
Other:
- moved on the sheet: C5
