File: version 2/v1/v1 4 button.brd (EAGLE design)
At the start: 45 x 63.5 mm, 31 parts, among them IC5 AMS1117-3.3V, X1 0446200002

Commit message: Add files via upload
Parts:
- added D1, D2, D3, D4: SM4007PL, SamacSys_Parts:SODFL3718X125N
- added J1: (no value), SparkFun-Connectors:SCREWTERMINAL-5MM-2
- added SJ1: (no value), SparkFun-Retired:SJ_3_PASTE1&2
- added U$2: LOGO, custom parts:LOGO
- C5: device rcl:UD-10X10_NICHICON -> SamacSys_Parts:CAPAE1030X1050N
- X1: device con-molex:0446200002 -> custom parts:0446200002
- moved C6 11.7 mm to (31.5, 48.5), turned to 270 degrees
- moved C7 11.5 mm to (34.5, 47.0), turned to 0 degrees
- moved C5 0.50 mm to (6.50, 55.0), turned to 270 degrees
Connections:
- new net D1-B1: D1.2, U$1.JP1.4
- new net D1-B2: D2.2, U$1.JP1.5
- new net D1-B3: D3.2, U$1.JP1.6
- new net D1-B4: D4.2, U$1.JP1.7
- new net N$17: SJ1.1, X1.4, X1.5
- new net N$18: J1.2, SJ1.3
- net B1: now also D1.1; no longer U$1.JP1.4
- net B2: now also D2.1; no longer U$1.JP1.5
- net B3: now also D3.1; no longer U$1.JP1.6
- net B4: now also D4.1; no longer U$1.JP1.7
- net GND: now also C5.2, J1.1; no longer C5.-
- net VCC: now also C5.1, IC5.4; no longer C5.+
- net VDD: now also SJ1.2; no longer X1.4, X1.5
Routing:
- net D1-B4: track 0.00 -> 31.0 mm
- net B4: track 77.6 -> 52.4 mm
- net B3: track 66.5 -> 52.5 mm, vias 2 -> 1
- net GND: track 119.8 -> 133.8 mm, vias 6 -> 5
- net N$18: track 0.00 -> 12.7 mm
- net N$17: track 0.00 -> 11.5 mm
- net D1-B3: track 0.00 -> 11.1 mm, vias 0 -> 1
- net D1-B1: track 0.00 -> 7.39 mm
- net D1-B2: track 0.00 -> 6.48 mm
- net VCC: track 339.6 -> 342.7 mm
- net B1: track 65.6 -> 68.0 mm
- net B2: track 87.7 -> 85.5 mm
- net VDD: track 23.3 -> 21.2 mm
- net LED: track 29.4 -> 31.3 mm, vias 2 -> 0
Other:
- board text added: "+ -"
- board text added: "7-30v"
- board text added: "V0.0.3"

Commit message: Add files via upload
Routing:
- net GND: track 133.8 -> 130.7 mm
Changed lines of the file:
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@@
 <contactref element="B2" pad="2"/>
 <contactref element="B3" pad="2"/>
-<wire x1="8.650003125" y1="56.150003125" x2="6.743303125" y2="50.593346875" width="1.27" layer="1"/>
 <wire x1="6.5" y1="50.35" x2="6.743303125" y2="50.593346875" width="1.27" layer="1"/>
-<wire x1="8" y1="54.5" x2="8" y2="55.5" width="1.27" layer="1"/>
-<wire x1="8.650003125" y1="56.150003125" x2="8" y2="55.5" width="1.27" layer="1"/>
 <via x="8" y="54.5" extent="1-16" drill="0.35"/>
 <wire x1="5.287865625" y1="35.11629375" x2="6.5" y2="36.328428125" width="1.016" layer="1"/>
@@
 <wire x1="34" y1="48.65" x2="34" y2="53" width="0.4064" layer="1"/>
 <wire x1="34" y1="53" x2="35.2006" y2="54.2006" width="0.4064" layer="1"/>
+<wire x1="6.5" y1="50.35" x2="6.5" y2="53" width="1.27" layer="1"/>
+<wire x1="6.5" y1="53" x2="8" y2="54.5" width="1.27" layer="1"/>
 <wire x1="32.11629375" y1="42.71213125" x2="31.5" y2="47.65" width="0" layer="19" extent="1-1"/>
 <wire x1="24.54" y1="53.04" x2="31.5" y2="47.65" width="0" layer="19" extent="1-1"/>
@@
 <wire x1="25.235" y1="6.4" x2="26.5" y2="6.4" width="0.4064" layer="16"/>
 </signal>
+<signal name="N$19">
+</signal>
 </signals>
